File: EAGLE Files/FINAL PROJECT.brd (EAGLE design)
At the start: 105.4 x 49.5 mm, 18 parts, among them J1 BATTERY, U1 9_to_3.3_VREG

Commit message: final EAGLE files
Parts:
- removed INT1: (no value), SparkFun-Connectors:1X01
- added J2: (no value), SparkFun-Connectors:1X01
- moved U1 3.81 mm to (16.5, 40.6)
- moved J1 3.81 mm to (6.35, 40.6)
- moved C3 3.81 mm to (24.1, 44.5)
- moved C4 3.81 mm to (24.1, 36.8)
- moved R1 3.81 mm to (14.1, 30.6)
- moved R2 3.81 mm to (25.4, 30.5)
- moved PSOC_PINS_1 2.54 mm to (90.2, 25.4)
- moved PSOC_PINS_2 2.54 mm to (34.3, 5.08)
- moved LED 2.54 mm to (92.7, 25.4)
- moved HC-05 1.27 mm to (105.3, 36.2)
Connections:
- removed net INT1: INT1.1, PSOC_PINS_1.9
Routing:
- net GND: track 301.8 -> 288.7 mm
- net INT1: track 12.2 -> 0.00 mm
- net 5V: track 22.3 -> 18.5 mm
- net VDD: track 82.7 -> 80.2 mm
- net LED: track 11.7 -> 9.20 mm
- net SCL: track 10.2 -> 11.2 mm
- net SCA: track 10.2 -> 11.2 mm
- net RX: track 7.04 -> 7.56 mm
Other:
- board size 105.4 x 49.5 mm -> 101.6 x 49.5 mm

Commit message: board
Parts:
- removed C3, C4: 0.1uF, SparkFun-Capacitors:CAP-PTH-SMALL-KIT
- removed PSOC_PINS_1: (no value), SparkFun-Connectors:1X13
- removed PSOC_PINS_2: (no value), SparkFun-Connectors:1X25
- removed R2: 1.5K, SparkFun-Resistors:AXIAL-0.3
- removed R3: 330, SparkFun-Resistors:AXIAL-0.3
- removed RED: (no value), SparkFun-LED:LED_3MM
- removed U1: 9_to_3.3_VREG, SparkFun-IC-Power:TO-92
- added C1: 0.33uF, SparkFun-Capacitors:CAP-PTH-SMALL-KIT
- added C2: 0.1uF, SparkFun-Capacitors:CAP-PTH-SMALL-KIT
- added D1: (no value), SparkFun-LED:LED_3MM
- added J3, J4, J5: (no value), SparkFun-Connectors:1X01
- added J6, J7: (no value), SparkFun-Connectors:1X02
- added U2: (no value), SparkFun-IC-Power:TO-220-ALT
- R1: value 1.2K -> 330
- moved R1 65.2 mm to (77.5, 45.7)
- moved J1 6.35 mm to (6.35, 34.3), turned to 90 degrees
Connections:
- removed net N$1: R3.P$2, RED.K
- removed net VDD: C3.1, CS.1, GND/VDD.2, HC-05.VCC, U1.1
- removed net VDD1: C4.1, J1.2, R1.P$2, U1.3
- new net 9V: C1.1, J1.2, U2.IN
- new net N$2: D1.K, R1.P$2
- net 5V: now also C2.1, CS.1, D1.A, GND/VDD.2, HC-05.VCC, U2.OUT; no longer R1.P$1, R2.P$2
- net GND: now also C1.2, C2.2, R1.P$1, U2.GND; no longer C3.2, C4.2, R2.P$1, R3.P$1, U1.2
- net LED: no longer RED.A
- net RX: now also J7.1; no longer PSOC_PINS_1.1
- net SCA: now also J6.1; no longer PSOC_PINS_1.12
- net SCL: now also J6.2; no longer PSOC_PINS_1.13
- net TX: now also J7.2; no longer PSOC_PINS_1.2
Routing:
- net GND: track 288.7 -> 201.0 mm
- net VDD: track 80.2 -> 0.00 mm
- net 5V: track 18.5 -> 94.8 mm
- net VDD1: track 27.2 -> 0.00 mm
- net 9V: track 0.00 -> 18.6 mm
- net LED: track 9.20 -> 0.00 mm
- net N$2: track 0.00 -> 3.81 mm
- net N$1: track 3.81 -> 0.00 mm
